File: DynamicRdsBoard.brd (EAGLE design)
At the start: 107.9 x 65.7 mm, 28 parts, among them Q1 FDP120N10, Q2 FDP120N10, U1 ADUM3223ARZ, X1 1751248, X2 1751280

Commit message: Friday work commit
Parts:
- added JP1: (no value), jumper:JP7Q
- added R10, R11, R5, R6, R7, R8, R9: 200 Thick Film, rcl:R1206
- R1: value 680m Thick Film -> 200 Thick Film; device rcl:R1210 -> rcl:R1206
Connections:
- new net N$2: JP1.2, R5.1
- new net N$3: JP1.4, R6.1
- new net N$4: JP1.6, R7.1
- new net N$5: JP1.8, R8.1
- new net N$6: JP1.10, R9.1
- new net N$7: JP1.12, R10.1
- new net N$8: JP1.14, R11.1
- net N$1: now also JP1.1, JP1.11, JP1.13, JP1.3, JP1.5, JP1.7, JP1.9
- net V+: now also R10.2, R11.2, R5.2, R6.2, R7.2, R8.2, R9.2
Routing:
- net N$1: track 23.3 -> 8.89 mm
